File: pretinhaMonitorBoard.sch (EAGLE design)
At the start: 14 parts

Commit message: Update
Parts:
- VIN+, VIN-, VOUT+, VOUT-: device pinhead:PINHD-1X1 -> adafruit:PINHD-1X1-BIGPOGO
Changed lines of the file:
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@@
 </variantdefs>
 <classes>
-<class number="0" name="default" width="0" drill="1">
-<clearance class="0" value="0.381"/>
+<class number="0" name="default" width="0.6" drill="1">
+<clearance class="0" value="0.2"/>
 </class>
 </classes>
@@
 <part name="GND6" library="supply1" library_urn="urn:adsk.eagle:library:371" deviceset="GND" device=""/>
 <part name="C1" library="SparkFun-Capacitors" library_urn="urn:adsk.eagle:library:510" deviceset="1000UF" device="-RADIAL-5MM-25V-20%" package3d_urn="urn:adsk.eagle:package:37412/1" value="1mF"/>
-<part name="VOUT-" library="pinhead" library_urn="urn:adsk.eagle:library:325" deviceset="PINHD-1X1" device="" package3d_urn="urn:adsk.eagle:package:22485/2"/>
-<part name="VOUT+" library="pinhead" library_urn="urn:adsk.eagle:library:325" deviceset="PINHD-1X1" device="" package3d_urn="urn:adsk.eagle:package:22485/2"/>
-<part name="VIN-" library="pinhead" library_urn="urn:adsk.eagle:library:325" deviceset="PINHD-1X1" device="" package3d_urn="urn:adsk.eagle:package:22485/2"/>
-<part name="VIN+" library="pinhead" library_urn="urn:adsk.eagle:library:325" deviceset="PINHD-1X1" device="" package3d_urn="urn:adsk.eagle:package:22485/2"/>
+<part name="VOUT-" library="adafruit" deviceset="PINHD-1X1" device="-BIGPOGO"/>
+<part name="VOUT+" library="adafruit" deviceset="PINHD-1X1" device="-BIGPOGO"/>
+<part name="VIN-" library="adafruit" deviceset="PINHD-1X1" device="-BIGPOGO"/>
+<part name="VIN+" library="adafruit" deviceset="PINHD-1X1" device="-BIGPOGO"/>
 <part name="GND7" library="supply1" library_urn="urn:adsk.eagle:library:371" deviceset="GND" device=""/>
 <part name="RPI" library="con-molex" library_urn="urn:adsk.eagle:library:165" deviceset="22-23-2021" device=""/>
